Commit message: add&modify world files and launch files

File: husky_ur3_gazebo/urdf/accessories/sick_tim571.urdf.xacro (robot description, xacro)
@@ -1,5 +1,5 @@
 <?xml version="1.0"?>
 <robot xmlns:xacro="http://www.ros.org/wiki/xacro">
-  <xacro:macro name="sensor_sick_tim571" params="prefix parent prefix_topic:='front_laser' *origin min_angle:=-1.57619449019 max_angle:=1.57619449019">
+  <xacro:macro name="sensor_sick_tim571" params="prefix parent topic *origin min_angle:=-1.57619449019 max_angle:=1.57619449019">
     <joint name="${prefix}_base_joint" type="fixed">
       <xacro:insert_block name="origin" />
@@ -62,5 +62,5 @@
 				</ray>
 				<plugin name="${prefix}_controller" filename="libgazebo_ros_laser.so">
-					<topicName>/scan</topicName>
+					<topicName>${topic}</topicName>
 					<frameName>/${prefix}_link</frameName>
 				</plugin>

File: husky_ur3_gazebo/urdf/decorations.urdf.xacro (robot description, xacro)
@@ -23,6 +23,6 @@
 <robot name="husky_decorations" xmlns:xacro="http://ros.org/wiki/xacro">
   <xacro:macro name="husky_decorate">
-    <xacro:property name="husky_front_bumper_extend" value="$(optenv HUSKY_FRONT_BUMPER_EXTEND 0)" />
-    <xacro:property name="husky_rear_bumper_extend" value="$(optenv HUSKY_REAR_BUMPER_EXTEND 0)" />
+    <xacro:property name="husky_front_bumper_extend" value="$(optenv HUSKY_FRONT_BUMPER_EXTEND 0.01)" />
+    <xacro:property name="husky_rear_bumper_extend" value="$(optenv HUSKY_REAR_BUMPER_EXTEND 0.01)" />
     <!-- Spawn Husky chassis -->
     <link name="top_chassis_link">
@@ -62,4 +62,9 @@
         </geometry>
       </visual>
+      <collision name="front_bumper_collision">
+        <geometry>
+          <mesh filename="package://husky_ur3_gazebo/meshes/bumper.dae" />
+        </geometry>
+      </collision>
     </link>
     <!-- Attach front bumper -->
@@ -90,4 +95,9 @@
         </geometry>
       </visual>
+      <collision name="rear_bumper_collision">
+        <geometry>
+          <mesh filename="package://husky_ur3_gazebo/meshes/bumper.dae" />
+        </geometry>
+      </collision>
     </link>
     <!-- Attach rear bumper -->

File: husky_ur3_gazebo/urdf/husky_ur3_gripper.urdf.xacro (robot description, xacro)
@@ -34,6 +34,6 @@
   <xacro:include filename="$(find husky_ur3_gazebo)/urdf/accessories/sick_tim571.urdf.xacro"/>
   <xacro:include filename="$(find husky_ur3_gazebo)/urdf/ur3_robot_gripper.urdf.xacro"/>
-  <xacro:include filename="$(find husky_ur3_gazebo)/urdf/accessories/d435_camera_h.urdf.xacro"/>-
-  <xacro:include filename="$(find husky_ur3_gazebo)/urdf/accessories/d435_camera_g.urdf.xacro"/>-
+  <xacro:include filename="$(find husky_ur3_gazebo)/urdf/accessories/d435_camera_h.urdf.xacro"/>
+  <!--xacro:include filename="$(find husky_ur3_gazebo)/urdf/accessories/d435_camera_g.urdf.xacro"/-->
   <!--xacro:include filename="$(find husky_ur3_gazebo)/urdf/ur3_robot.urdf.xacro"/-->
   <xacro:property name="M_PI" value="3.14159"/>
@@ -57,14 +57,14 @@
       </geometry>
     </visual>
-    <collision>
+    <collision name = "base_collision1">
       <origin xyz="${( husky_front_bumper_extend - husky_rear_bumper_extend ) / 2.0} 0 ${base_z_size/4}" rpy="0 0 0" />
       <geometry>
-        <box size="${ base_x_size + husky_front_bumper_extend + husky_rear_bumper_extend } ${base_y_size} ${base_z_size/2}"/>
+        <box size="${ base_x_size + husky_front_bumper_extend + husky_rear_bumper_extend } ${base_y_size + 0.12} ${base_z_size/2}"/>
       </geometry>
     </collision>
-    <collision>
+    <collision name = "base_collision2">
       <origin xyz="0 0 ${base_z_size*3/4-0.01}" rpy="0 0 0" />
       <geometry>
-        <box size="${base_x_size*4/5} ${base_y_size} ${base_z_size/2-0.02}"/>
+        <box size="${base_x_size*4/5} ${base_y_size + 0.12} ${base_z_size/2-0.02}"/>
       </geometry>
     </collision>
@@ -150,5 +150,5 @@
 	</gazebo>
   <xacro:husky_decorate />
-  <xacro:sensor_sick_tim571 prefix="front_laser" parent="top_plate_link" prefix_topic="front_laser">
+  <xacro:sensor_sick_tim571 prefix="front_laser" parent="top_plate_link" topic="scan">
    	<origin xyz="$(arg laser_xyz)" rpy="$(arg laser_rpy)"/>
   </xacro:sensor_sick_tim571>
@@ -217,4 +217,64 @@
     </plugin>
   </gazebo>
+  <gazebo>
+    <plugin name="p3d_base_controller" filename="libgazebo_ros_p3d.so">
+      <alwaysOn>true</alwaysOn>
+      <updateRate>50.0</updateRate>
+      <bodyName>base_footprint</bodyName>
+      <topicName>base_pose_ground_truth</topicName>
+      <gaussianNoise>0.01</gaussianNoise>
+      <frameName>map</frameName>
+      <xyzOffsets>0 0 0</xyzOffsets>
+      <rpyOffsets>0 0 0</rpyOffsets>
+    </plugin>
+  </gazebo>
+  <gazebo reference="base_link">
+      <!-- Virtual Contact Sensor -->
+      <sensor name='base_contact_sensor' type='contact'>
+         <contact>
+             <collision>base_link_fixed_joint_lump__base_collision1_collision</collision>
+         </contact>
+         <plugin name="my_plugin" filename="libgazebo_ros_bumper.so">
+            <bumperTopicName>husky_collision</bumperTopicName>
+            <frameName>base_link</frameName>
+         </plugin>
+      </sensor>
+   </gazebo>
+   <gazebo reference="base_link">
+      <!-- Virtual Contact Sensor -->
+      <sensor name='base_contact_sensor2' type='contact'>
+         <contact>
+             <collision>base_link_fixed_joint_lump__base_collision2_collision_1</collision>
+         </contact>
+         <plugin name="my_plugin2" filename="libgazebo_ros_bumper.so">
+            <bumperTopicName>husky_collision</bumperTopicName>
+            <frameName>base_link</frameName>
+         </plugin>
+      </sensor>
+   </gazebo>
+    <gazebo reference="rear_bumper_link">
+      <!-- Virtual Contact Sensor -->
+      <sensor name='base_contact_sensor3' type='contact'>
+         <contact>
+             <collision>base_link_fixed_joint_lump__rear_bumper_collision_collision_3</collision>
+         </contact>
+         <plugin name="my_plugin3" filename="libgazebo_ros_bumper.so">
+            <bumperTopicName>husky_collision</bumperTopicName>
+            <frameName>base_link</frameName>
+         </plugin>
+      </sensor>
+   </gazebo>
+    <gazebo reference="front_bumper_link">
+      <!-- Virtual Contact Sensor -->
+      <sensor name='base_contact_sensor4' type='contact'>
+         <contact>
+             <collision>base_link_fixed_joint_lump__front_bumper_collision_collision_2</collision>
+         </contact>
+         <plugin name="my_plugin4" filename="libgazebo_ros_bumper.so">
+            <bumperTopicName>husky_collision</bumperTopicName>
+            <frameName>base_link</frameName>
+         </plugin>
+      </sensor>
+   </gazebo>
   <!-- Optional custom includes. -->
   <xacro:include filename="$(arg urdf_extras)" />

Commit message: modify scan sensor plugin reflected real robot lidar specification

File: husky_ur3_gazebo/urdf/accessories/sick_tim571.urdf.xacro (robot description, xacro)
@@ -1,5 +1,5 @@
 <?xml version="1.0"?>
 <robot xmlns:xacro="http://www.ros.org/wiki/xacro">
-  <xacro:macro name="sensor_sick_tim571" params="prefix parent topic *origin min_angle:=-1.57619449019 max_angle:=1.57619449019">
+  <xacro:macro name="sensor_sick_tim571" params="prefix parent topic *origin min_angle:=-1.757025 max_angle:=1.756554">
     <joint name="${prefix}_base_joint" type="fixed">
       <xacro:insert_block name="origin" />
@@ -44,5 +44,5 @@
 					<scan>
 						<horizontal>
-							<samples>716</samples>
+							<samples>542</samples>
 							<resolution>1</resolution>
 							<min_angle>${min_angle}</min_angle>

Commit message: sick tim571 sensor angular modified

File: husky_ur3_gazebo/urdf/accessories/sick_tim571.urdf.xacro (robot description, xacro)
@@ -1,5 +1,5 @@
 <?xml version="1.0"?>
 <robot xmlns:xacro="http://www.ros.org/wiki/xacro">
-  <xacro:macro name="sensor_sick_tim571" params="prefix parent topic *origin min_angle:=-1.757025 max_angle:=1.756554">
+  <xacro:macro name="sensor_sick_tim571" params="prefix parent topic *origin min_angle:=-1.57 max_angle:=1.57">
     <joint name="${prefix}_base_joint" type="fixed">
       <xacro:insert_block name="origin" />
@@ -40,5 +40,5 @@
 				<pose>0 0 0 0 0 0</pose>
 				<visualize>false</visualize>
-				<update_rate>15</update_rate>
+				<update_rate>30</update_rate>
 				<ray>
 					<scan>

Commit message: add some collision sensors

File: husky_ur3_gazebo/urdf/accessories/sick_tim571.urdf.xacro (robot description, xacro)
@@ -55,9 +55,9 @@
 						<resolution>0.00575</resolution>
 					</range>
-					<noise>
+					<!-- <noise>
 						<type>gaussian</type>
 						<mean>0.0</mean>
 						<stddev>0.01</stddev>
-					</noise>
+					</noise> -->
 				</ray>
 				<plugin name="${prefix}_controller" filename="libgazebo_ros_laser.so">

File: husky_ur3_gazebo/urdf/decorations.urdf.xacro (robot description, xacro)
@@ -194,4 +194,140 @@
       <link name="top_plate_rear_link"/>
     </xacro:if>
+ <joint name="side_bumper_joint" type="fixed">
+      <origin xyz="-0.2 -0.6 0.085" rpy="${M_PI/2} 0 0" />
+      <parent link="top_plate_link"/>
+      <child link="side_bumper_link" />
+    </joint>
+  <link name="side_bumper_link">
+    <inertial>
+      <mass value="5.0" />
+      <origin xyz="0 0 0" />
+      <inertia  ixx="0.0" ixy="0.0"  ixz="0.0"  iyy="0.0"  iyz="0.0"  izz="0.0" />
+    </inertial>
+    <!-- <visual>
+       <origin xyz="0 0 0" rpy="0 -${M_PI/2} 0 " />
+       <geometry>
+           <box size="0.003 0.8 0.83"/>
+       </geometry>
+       <material name="gray">
+         <color rgba="0.153 0.153 0.153 1"/>
+       </material>
+    </visual>   -->
+    <collision name="side_bumper_link">
+       <origin xyz="0 0 0" rpy="0 -${M_PI/2} 0 " />
+       <geometry>
+           <box size="0.003 0.8 1.0"/>
+       </geometry>
+    </collision>
+  </link>
+ <joint name="side_bumper_joint2" type="fixed">
+      <origin xyz="-0.2 0.6 0.085" rpy="${M_PI/2} 0 0" />
+      <parent link="top_plate_link"/>
+      <child link="side_bumper_link2" />
+    </joint>
+  <link name="side_bumper_link2">
+    <inertial>
+      <mass value="5.0" />
+      <origin xyz="0 0 0" />
+      <inertia  ixx="0.0" ixy="0.0"  ixz="0.0"  iyy="0.0"  iyz="0.0"  izz="0.0" />
+    </inertial>
+    <!-- <visual>
+       <origin xyz="0 0 0" rpy="0 -${M_PI/2} 0 " />
+       <geometry>
+           <box size="0.003 0.8 0.83"/>
+       </geometry>
+       <material name="gray">
+         <color rgba="0.153 0.153 0.153 1"/>
+       </material>
+    </visual>   -->
+    <collision name="side_bumper_link2">
+       <origin xyz="0 0 0" rpy="0 -${M_PI/2} 0 " />
+       <geometry>
+           <box size="0.003 0.8 1.0"/>
+       </geometry>
+    </collision>
+  </link>
+    <!-- add more bumper collision -->
+  <joint name="another_bumper_joint" type="fixed">
+        <origin xyz="0.09 0 -0.05" rpy="0 0 0" />
+        <parent link="front_bumper_link"/>
+        <child link="another_bumper_link" />
+  </joint>
+    <link name="another_bumper_link">
+      <inertial>
+        <mass value="5.0" />
+        <origin xyz="0 0 0" />
+        <inertia  ixx="0.0" ixy="0.0"  ixz="0.0"  iyy="0.0"  iyz="0.0"  izz="0.0" />
+      </inertial>
+      <!-- <visual>
+        <origin xyz="0 0 0" rpy="0 -${M_PI/2} 0 " />
+        <geometry>
+            <box size="0.05 0.7 0.005"/>
+        </geometry>
+        <material name="gray">
+          <color rgba="0.153 0.153 0.153 1"/>
+        </material>
+      </visual>   -->
+      <collision name="another_bumper_link">
+        <origin xyz="0 0 0" rpy="0 -${M_PI/2} 0 " />
+        <geometry>
+            <box size="0.25 1.0 0.003"/>
+        </geometry>
+      </collision>
+    </link>
+  <joint name="another_bumper_joint2" type="fixed">
+    <origin xyz="0.09 0 0.30" rpy="0 0 0" />
+    <parent link="rear_bumper_link"/>
+    <child link="another_bumper_link2" />
+  </joint>
+    <link name="another_bumper_link2">
+      <inertial>
+        <mass value="5.0" />
+        <origin xyz="0 0 0" />
+        <inertia  ixx="0.0" ixy="0.0"  ixz="0.0"  iyy="0.0"  iyz="0.0"  izz="0.0" />
+      </inertial>
+      <!-- <visual>
+        <origin xyz="0 0 0" rpy="0 -${M_PI/2} 0 " />
+        <geometry>
+            <box size="0.05 0.7 0.005"/>
+        </geometry>
+        <material name="gray">
+          <color rgba="0.153 0.153 0.153 1"/>
+        </material>
+      </visual>   -->
+      <collision name="another_bumper_link2">
+        <origin xyz="0 0 0" rpy="0 -${M_PI/2} 0 " />
+        <geometry>
+            <box size="1.0 1.0 0.003"/>
+        </geometry>
+      </collision>
+    </link>
+  <joint name="another_bumper_joint3" type="fixed">
+    <origin xyz="0.09 0 0.5" rpy="0 0 0" />
+    <parent link="front_bumper_link"/>
+    <child link="another_bumper_link3" />
+  </joint>
+    <link name="another_bumper_link3">
+      <inertial>
+        <mass value="5.0" />
+        <origin xyz="0 0 0" />
+        <inertia  ixx="0.0" ixy="0.0"  ixz="0.0"  iyy="0.0"  iyz="0.0"  izz="0.0" />
+      </inertial>
+      <!-- <visual>
+        <origin xyz="0 0 0" rpy="0 -${M_PI/2} 0 " />
+        <geometry>
+            <box size="0.05 0.7 0.005"/>
+        </geometry>
+        <material name="gray">
+          <color rgba="0.153 0.153 0.153 1"/>
+        </material>
+      </visual>   -->
+      <collision name="another_bumper_link3">
+        <origin xyz="0 0 0" rpy="0 -${M_PI/2} 0 " />
+        <geometry>
+            <box size="0.6 1.0 0.003"/>
+        </geometry>
+      </collision>
+    </link>
     <!--D435 mount frame -->
     <!--<link name="mount_link">

File: husky_ur3_gazebo/urdf/husky_ur3_gripper.urdf.xacro (robot description, xacro)
@@ -180,4 +180,58 @@
     </collision>
   </link>
+ <!-- <joint name="control_box_ur3_joint2" type="fixed">
+      <origin xyz="-0.095 -0.36 0.233" rpy="${M_PI/2} 0 0" />
+      <parent link="top_plate_link"/>
+      <child link="control_box_ur3_link2" />
+    </joint>
+  <link name="control_box_ur3_link2">
+    <inertial>
+      <mass value="5.0" />
+      <origin xyz="0 0 0" />
+      <inertia  ixx="0.0" ixy="0.0"  ixz="0.0"  iyy="0.0"  iyz="0.0"  izz="0.0" />
+    </inertial>
+    <visual>
+       <origin xyz="0 0 0" rpy="0 -${M_PI/2} 0 " />
+       <geometry>
+           <box size="0.003 0.8 0.85"/>
+       </geometry>
+       <material name="gray">
+         <color rgba="0.153 0.153 0.153 1"/>
+       </material>
+    </visual>
+    <collision>
+       <origin xyz="0 0 0" rpy="0 -${M_PI/2} 0 " />
+       <geometry>
+           <box size="0.003 0.8 0.85"/>
+       </geometry>
+    </collision>
+  </link>
+ <joint name="control_box_ur3_joint3" type="fixed">
+      <origin xyz="-0.095 0.36 0.233" rpy="${M_PI/2} 0 0" />
+      <parent link="top_plate_link"/>
+      <child link="control_box_ur3_link3" />
+    </joint>
+  <link name="control_box_ur3_link3">
+    <inertial>
+      <mass value="5.0" />
+      <origin xyz="0 0 0" />
+      <inertia  ixx="0.0" ixy="0.0"  ixz="0.0"  iyy="0.0"  iyz="0.0"  izz="0.0" />
+    </inertial>
+    <visual>
+       <origin xyz="0 0 0" rpy="0 -${M_PI/2} 0 " />
+       <geometry>
+           <box size="0.003 0.8 0.85"/>
+       </geometry>
+       <material name="gray">
+         <color rgba="0.153 0.153 0.153 1"/>
+       </material>
+    </visual>
+    <collision>
+       <origin xyz="0 0 0" rpy="0 -${M_PI/2} 0 " />
+       <geometry>
+           <box size="0.003 0.8 0.85"/>
+       </geometry>
+    </collision>
+  </link> -->
   <gazebo reference="control_box_ur3_link">
     <material>Gazebo/DarkGrey</material>
@@ -231,50 +285,121 @@
   <gazebo reference="base_link">
       <!-- Virtual Contact Sensor -->
-      <sensor name='base_contact_sensor' type='contact'>
+      <sensor name='base_contact_sensor3' type='contact'>
          <contact>
              <collision>base_link_fixed_joint_lump__base_collision1_collision</collision>
          </contact>
-         <plugin name="my_plugin" filename="libgazebo_ros_bumper.so">
+         <plugin name="my_plugin3" filename="libgazebo_ros_bumper.so">
             <bumperTopicName>husky_collision</bumperTopicName>
             <frameName>base_link</frameName>
          </plugin>
+         <update_rate>5</update_rate>
       </sensor>
    </gazebo>
    <gazebo reference="base_link">
       <!-- Virtual Contact Sensor -->
-      <sensor name='base_contact_sensor2' type='contact'>
+      <sensor name='base_contact_sensor4' type='contact'>
          <contact>
              <collision>base_link_fixed_joint_lump__base_collision2_collision_1</collision>
          </contact>
-         <plugin name="my_plugin2" filename="libgazebo_ros_bumper.so">
+         <plugin name="my_plugin4" filename="libgazebo_ros_bumper.so">
             <bumperTopicName>husky_collision</bumperTopicName>
             <frameName>base_link</frameName>
          </plugin>
+         <update_rate>5</update_rate>
+      </sensor>
+   </gazebo>
+    <gazebo reference="front_bumper_link">
+      <!-- Virtual Contact Sensor -->
+      <sensor name='base_contact_sensor' type='contact'>
+         <contact>
+             <collision>base_link_fixed_joint_lump__front_bumper_collision_collision_2</collision>
+         </contact>
+         <plugin name="my_plugin" filename="libgazebo_ros_bumper.so">
+            <bumperTopicName>husky_collision</bumperTopicName>
+            <frameName>base_link</frameName>
+         </plugin>
+         <update_rate>5</update_rate>
       </sensor>
    </gazebo>
     <gazebo reference="rear_bumper_link">
       <!-- Virtual Contact Sensor -->
-      <sensor name='base_contact_sensor3' type='contact'>
-         <contact>
-             <collision>base_link_fixed_joint_lump__rear_bumper_collision_collision_3</collision>
-         </contact>
-         <plugin name="my_plugin3" filename="libgazebo_ros_bumper.so">
+      <sensor name='base_contact_sensor2' type='contact'>
+         <contact>
+             <collision>base_link_fixed_joint_lump__rear_bumper_collision_collision_5</collision>
+         </contact>
+         <plugin name="my_plugin2" filename="libgazebo_ros_bumper.so">
             <bumperTopicName>husky_collision</bumperTopicName>
             <frameName>base_link</frameName>
          </plugin>
+         <update_rate>5</update_rate>
       </sensor>
    </gazebo>
-    <gazebo reference="front_bumper_link">
-      <!-- Virtual Contact Sensor -->
-      <sensor name='base_contact_sensor4' type='contact'>
-         <contact>
-             <collision>base_link_fixed_joint_lump__front_bumper_collision_collision_2</collision>
-         </contact>
-         <plugin name="my_plugin4" filename="libgazebo_ros_bumper.so">
-            <bumperTopicName>husky_collision</bumperTopicName>
-            <frameName>base_link</frameName>
-         </plugin>
-      </sensor>
-   </gazebo>
+<!--ADD-->
+  <gazebo reference="side_bumper_link">
+      <!-- Virtual Contact Sensor -->
+      <sensor name='control_box_contact_sensor' type='contact'>
+         <contact>
+             <collision>base_link_fixed_joint_lump__side_bumper_link_collision_12</collision>
+         </contact>
+         <plugin name="my_plugin5" filename="libgazebo_ros_bumper.so">
+            <bumperTopicName>husky_collision</bumperTopicName>
+            <frameName>top_plate_link</frameName>
+         </plugin>
+         <update_rate>5</update_rate>
+      </sensor>
+  </gazebo>
+  <gazebo reference="side_bumper_link2">
+      <!-- Virtual Contact Sensor -->
+      <sensor name='control_box_contact_sensor2' type='contact'>
+         <contact>
+             <collision>base_link_fixed_joint_lump__side_bumper_link2_collision_13</collision>
+         </contact>
+         <plugin name="my_plugin6" filename="libgazebo_ros_bumper.so">
+            <bumperTopicName>husky_collision</bumperTopicName>
+            <frameName>top_plate_link</frameName>
+         </plugin>
+         <update_rate>5</update_rate>
+      </sensor>
+  </gazebo>
+<!--ADD 2-->
+  <gazebo reference="another_bumper_link">
+      <!-- Virtual Contact Sensor -->
+      <sensor name='base_contact_sensor5' type='contact'>
+         <contact>
+             <collision>base_link_fixed_joint_lump__another_bumper_link_collision_3</collision>
+         </contact>
+         <plugin name="my_plugin7" filename="libgazebo_ros_bumper.so">
+            <bumperTopicName>husky_collision</bumperTopicName>
+            <frameName>front_bumper_link</frameName>
+         </plugin>
+         <update_rate>5</update_rate>
+      </sensor>
+  </gazebo>
+  <gazebo reference="another_bumper_link2">
+      <!-- Virtual Contact Sensor -->
+      <sensor name='base_contact_sensor6' type='contact'>
+         <contact>
+             <collision>base_link_fixed_joint_lump__another_bumper_link2_collision_6</collision>
+         </contact>
+         <plugin name="my_plugin8" filename="libgazebo_ros_bumper.so">
+            <bumperTopicName>husky_collision</bumperTopicName>
+            <frameName>rear_bumper_link</frameName>
+         </plugin>
+         <update_rate>5</update_rate>
+      </sensor>
+  </gazebo>
+  <gazebo reference="another_bumper_link3">
+      <!-- Virtual Contact Sensor -->
+      <sensor name='base_contact_sensor7' type='contact'>
+         <contact>
+             <collision>base_link_fixed_joint_lump__another_bumper_link3_collision_4</collision>
+         </contact>
+         <plugin name="my_plugin8" filename="libgazebo_ros_bumper.so">
+            <bumperTopicName>husky_collision</bumperTopicName>
+            <frameName>front_bumper_link</frameName>
+         </plugin>
+         <update_rate>5</update_rate>
+      </sensor>
+  </gazebo>
   <!-- Optional custom includes. -->
   <xacro:include filename="$(arg urdf_extras)" />
